File: Hardware/Electronics/CAD/LightSwitch.kicad_pcb (KiCad board)
At the start: 2 copper layers, 37.1 x 36.4 mm, 17 parts, among them J1 MPE 094-1-006, J2 MPE 087-1-002, J3 MPE 087-1-002, J4 RND 205-00232, J5 RND 205-00232, J6 RND 205-00232, J7 CONN_01X03, SW2 SW_DPST_x2, U1 IXYS CPC1966Y, U2 IXYS CPC1966Y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

Commit message: 3d model improvement and default parts
Parts:
- J4, J5, J6: footprint WAGO:WAGO_2pin -> Terminal:WAGO_2pin
- J7: value CONN_01X03 -> MPE 087-1-003
- SW2: value SW_DPST_x2 -> TASTER 9314
- U3: footprint HiLink:HiLink -> HiLink:HLK-PM01
