File: Hardware/Electronics/CAD/LightSwitch.kicad_pcb (KiCad board)
At the start: 2 copper layers, 37.1 x 36.4 mm, 17 parts, among them J1 MPE 094-1-006, J2 MPE 087-1-002, J3 MPE 087-1-002, J4 RND 205-00232, J5 RND 205-00232, J6 RND 205-00232, J7 MPE 087-1-003, SW2 TASTER 9314, U1 IXYS CPC1966Y, U2 IXYS CPC1966Y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

Commit message: library linkage fix
Parts:
- SW2: value TASTER 9314 -> SMD 4x4mm Button
Changed lines of the file:
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@@
       (effects (font (size 1 1) (thickness 0.15)))
     )
-    (fp_text value "TASTER 9314" (at 0 3.75 180) (layer F.Fab)
+    (fp_text value "SMD 4x4mm Button" (at 0 3.75 180) (layer F.Fab)
       (effects (font (size 1 1) (thickness 0.15)))
     )

Commit message: terminal footprints
Parts:
- J4, J5, J6: footprint Terminal:WAGO_2pin -> Terminal:Terminal_1x2_2.54mm
Changed lines of the file:
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@@
     )
   )
-  (module Terminal:WAGO_2pin (layer F.Cu)
+  (module HiLink:HLK-PM01 (layer F.Cu)
+    (at 147.32 124.46)
+    (fp_text reference U3 (at 0 0.5) (layer F.SilkS)
+      (effects (font (size 1 1) (thickness 0.15)))
+    )
+    (fp_text value HLK-PM05 (at 0 -1.27) (layer F.Fab)
+      (effects (font (size 1 1) (thickness 0.15)))
+    )
+    (fp_line (start -17 -10.1) (end 17 -10.1) (layer F.SilkS) (width 0.15))
+    (fp_line (start 17 -10.1) (end 17 10.1) (layer F.SilkS) (width 0.15))
+    (fp_line (start 17 10.1) (end -17 10.1) (layer F.SilkS) (width 0.15))
+    (fp_line (start -17 10.1) (end -17 -10.1) (layer F.SilkS) (width 0.15))
+    (pad 1 thru_hole circle (at -14.7 -2.5) (size 1.524 1.524) (drill 0.762) (layers *.Cu *.Mask)
+      (net 13 "Net-(J6-Pad2)"))
+    (pad 2 thru_hole circle (at -14.7 2.5) (size 1.524 1.524) (drill 0.762) (layers *.Cu *.Mask)
+      (net 14 "Net-(J6-Pad1)"))
+    (pad 3 thru_hole circle (at 14.7 -7.7) (size 1.524 1.524) (drill 0.762) (layers *.Cu *.Mask)
+      (net 1 GND))
+    (pad 4 thru_hole circle (at 14.7 7.7) (size 1.524 1.524) (drill 0.762) (layers *.Cu *.Mask)
+      (net 2 +3V3))
+    (model ${KIPRJMOD}/Libraries/3DParts/HiLink.3dshapes/HiLinkHLK-PM01.wrl
+      (at (xyz -0.669291 -0.397638 0))
+      (scale (xyz 0.3937 0.3937 0.3937))
+      (rotate (xyz 0 0 0))
+    )
+  )
+  (module Terminal:Terminal_1x2_2.54mm (layer F.Cu)
     (at 135.509 101.473 180)
     (fp_text reference J6 (at 0.127 -1.778 180) (layer F.SilkS)
@@
     )
   )
-  (module Terminal:WAGO_2pin (layer F.Cu)
+  (module Terminal:Terminal_1x2_2.54mm (layer F.Cu)
     (at 149.098 101.4984 180)
     (fp_text reference J5 (at 0.127 -1.778 180) (layer F.SilkS)
@@
     )
   )
-  (module Terminal:WAGO_2pin (layer F.Cu)
+  (module Terminal:Terminal_1x2_2.54mm (layer F.Cu)
     (at 159.258 101.473 180)
     (fp_text reference J4 (at 0.127 -1.778 180) (layer F.SilkS)
@@
       (rotate (xyz 0 0 0))
     )
-  )
-  (module HiLink:HLK-PM01 (layer F.Cu)
-    (at 147.32 124.46)
-    (fp_text reference U3 (at 0 0.5) (layer F.SilkS)
-      (effects (font (size 1 1) (thickness 0.15)))
-    )
-    (fp_text value HLK-PM05 (at 0 -1.27) (layer F.Fab)
-      (effects (font (size 1 1) (thickness 0.15)))
-    )
-    (fp_line (start -17 -10.1) (end 17 -10.1) (layer F.SilkS) (width 0.15))
-    (fp_line (start 17 -10.1) (end 17 10.1) (layer F.SilkS) (width 0.15))
-    (fp_line (start 17 10.1) (end -17 10.1) (layer F.SilkS) (width 0.15))
-    (fp_line (start -17 10.1) (end -17 -10.1) (layer F.SilkS) (width 0.15))
-    (pad 1 thru_hole circle (at -14.7 -2.5) (size 1.524 1.524) (drill 0.762) (layers *.Cu *.Mask)
-      (net 13 "Net-(J6-Pad2)"))
-    (pad 2 thru_hole circle (at -14.7 2.5) (size 1.524 1.524) (drill 0.762) (layers *.Cu *.Mask)
-      (net 14 "Net-(J6-Pad1)"))
-    (pad 3 thru_hole circle (at 14.7 -7.7) (size 1.524 1.524) (drill 0.762) (layers *.Cu *.Mask)
-      (net 1 GND))
-    (pad 4 thru_hole circle (at 14.7 7.7) (size 1.524 1.524) (drill 0.762) (layers *.Cu *.Mask)
-      (net 2 +3V3))
-    (model ${KIPRJMOD}/Libraries/3DParts/HiLink.3dshapes/HiLinkHLK-PM01.wrl
-      (at (xyz -0.669291 -0.397638 0))
-      (scale (xyz 0.3937 0.3937 0.3937))
-      (rotate (xyz 0 0 0))
-    )

Commit message: documentation
Other:
- board text added: "Home Automation Switch + Relay Revision 1.2.0 by Felix Kübler"
- board text removed: "Home Automation Switch + Relay Revision 1.0.2 by Felix Kübler"
Changed lines of the file:
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@@
     (links 38)
     (no_connects 2)
-    (area 127.178999 98.095999 164.413001 134.695001)
+    (area 112.54681 90.01 180.951 138.265)
     (thickness 1.6)
     (drawings 8)
@@
   (title_block
     (title "Light Switch")
-    (date 2018-02-10)
-    (rev 1.1.0)
+    (date 2018-09-20)
+    (rev 1.2.0)
     (company "Felix Kübler")
   )
@@
       (padsonsilk false)
       (subtractmaskfromsilk false)
-      (outputformat 4)
+      (outputformat 1)
       (mirror false)
       (drillshape 0)
       (scaleselection 1)
-      (outputdirectory ../Plots/))
+      (outputdirectory ../Gerber/))
   )
   (net 0 "")
@@
     )
   )
-  (gr_text "Home Automation\nSwitch + Relay\nRevision 1.0.2\nby Felix Kübler" (at 134.493 104.267 90) (layer B.SilkS)
+  (gr_text "Home Automation\nSwitch + Relay\nRevision 1.2.0\nby Felix Kübler" (at 134.493 104.267 90) (layer B.SilkS)
     (effects (font (size 0.8 0.8) (thickness 0.15)) (justify left mirror))
   )
