File: Hardware/Electronics/CAD/LightSwitch.sch (KiCad schematic (older format))
At the start: 17 parts, among them J1 MPE 094-1-006, J2 MPE 087-1-002, J3 MPE 087-1-002, J4 RND 205-00232, J5 RND 205-00232, J6 RND 205-00232, J7 CONN_01X03, SW2 SW_DPST_x2, U1 IXYS CPC1966Y, U2 IXYS CPC1966Y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

Commit message: 3d model improvement and default parts
Parts:
- J4, J5, J6: footprint WAGO:WAGO_2pin_5.0 -> Terminal:WAGO_2pin
- J7: value CONN_01X03 -> MPE 087-1-003
- SW2: value SW_DPST_x2 -> TASTER 9314
- U1, U2: footprint SharpSSR:SharpSSR -> SSR:CPC1966Y
- U3: footprint HiLink:HiLink -> HiLink:HLK-PM01
Changed lines of the file:
@@
 F 0 "U3" H 7250 1775 60  0000 C CNN
 F 1 "HLK-PM05" H 7425 1700 60  0000 C CNN
-F 2 "HiLink:HiLink" H 7425 1475 60  0001 C CNN
+F 2 "HiLink:HLK-PM01" H 7425 1475 60  0001 C CNN
 F 3 "" H 7425 1475 60  0001 C CNN
 	1    7425 1475
@@
 F 0 "J6" H 6800 1175 50  0000 C TNN
 F 1 "RND 205-00232" H 6525 1275 50  0000 C TNN
-F 2 "WAGO:WAGO_2pin_5.0" H 6725 1250 50  0001 C CNN
+F 2 "Terminal:WAGO_2pin" H 6725 1250 50  0001 C CNN
 F 3 "" H 6700 1475 50  0001 C CNN
 	1    6725 1475
@@
 F 0 "J5" H 3950 6000 50  0000 C TNN
 F 1 "RND 205-00232" H 3675 6075 50  0000 C TNN
-F 2 "WAGO:WAGO_2pin_5.0" H 3900 6050 50  0001 C CNN
+F 2 "Terminal:WAGO_2pin" H 3900 6050 50  0001 C CNN
 F 3 "" H 3875 6275 50  0001 C CNN
 	1    3900 6275
@@
 F 0 "U2" H 3000 6600 60  0000 C CNN
 F 1 "IXYS CPC1966Y" H 3300 6525 60  0000 C CNN
-F 2 "SharpSSR:SharpSSR" H 3375 6275 60  0001 C CNN
+F 2 "SSR:CPC1966Y" H 3375 6275 60  0001 C CNN
 F 3 "" H 3375 6275 60  0001 C CNN
 	1    3250 6275
@@
 F 0 "J4" H 3950 5975 50  0000 C TNN
 F 1 "RND 205-00232" H 3675 5900 50  0000 C TNN
-F 2 "WAGO:WAGO_2pin_5.0" H 3900 5400 50  0001 C CNN
+F 2 "Terminal:WAGO_2pin" H 3900 5400 50  0001 C CNN
 F 3 "" H 3875 5625 50  0001 C CNN
 	1    3900 5625
@@
 F 0 "U1" H 3000 5950 60  0000 C CNN
 F 1 "IXYS CPC1966Y" H 3300 5875 60  0000 C CNN
-F 2 "SharpSSR:SharpSSR" H 3375 5625 60  0001 C CNN
+F 2 "SSR:CPC1966Y" H 3375 5625 60  0001 C CNN
 F 3 "" H 3375 5625 60  0001 C CNN
 	1    3250 5625
@@
 P 7050 2500
 F 0 "SW2" H 7050 2400 50  0000 C CNN
-F 1 "SW_DPST_x2" H 7050 2300 50  0000 C CNN
+F 1 "TASTER 9314" H 7050 2300 50  0000 C CNN
 F 2 "Buttons_Switches_SMD:SW_SPST_TL3342" H 7050 2500 50  0001 C CNN
 F 3 "" H 7050 2500 50  0001 C CNN
@@
 P 7600 2650
 F 0 "R5" V 7680 2650 50  0000 C CNN
-F 1 "RND 0805 1 10K" V 7750 2650 50  0000 C CNN
+F 1 "RND 0805 1 10K" V 7750 2925 50  0000 C CNN
 F 2 "Resistors_SMD:R_0805" V 7530 2650 50  0001 C CNN
 F 3 "" H 7600 2650 50  0001 C CNN
@@
 P 2725 2800
 F 0 "J7" H 2725 2500 50  0000 C CNN
-F 1 "CONN_01X03" H 2725 2575 50  0000 C CNN
+F 1 "MPE 087-1-003" H 3000 2575 50  0000 C CNN
 F 2 "Pin_Headers:Pin_Header_Straight_1x03_Pitch2.54mm" H 2725 2800 50  0001 C CNN
 F 3 "" H 2725 2800 50  0001 C CNN

Commit message: library linkage fix
Parts:
- SW2: value TASTER 9314 -> SMD 4x4mm Button
Connections:
- net reset: now also SW2.2
Other:
- moved on the sheet: SW2
Changed lines of the file:
@@
 LIBS:HiLink
 LIBS:SharpSSR
-LIBS:LightSwitch-cache
+LIBS:SW_DPST_x2
 EELAYER 25 0
 EELAYER END
@@
 L SW_DPST_x2 SW2
 U 1 1 599EBC5A
-P 7050 2500
-F 0 "SW2" H 7050 2400 50  0000 C CNN
-F 1 "TASTER 9314" H 7050 2300 50  0000 C CNN
-F 2 "Buttons_Switches_SMD:SW_SPST_TL3342" H 7050 2500 50  0001 C CNN
-F 3 "" H 7050 2500 50  0001 C CNN
-	1    7050 2500
+P 6900 2500
+F 0 "SW2" H 6900 2400 50  0000 C CNN
+F 1 "SMD 4x4mm Button" H 6900 2300 50  0000 C CNN
+F 2 "Buttons_Switches_SMD:SW_SPST_TL3342" H 6900 2500 50  0001 C CNN
+F 3 "" H 6900 2500 50  0001 C CNN
+	1    6900 2500
 	1    0    0    -1
 $EndComp
@@
 L +3.3V #PWR015
 U 1 1 599EBD49
-P 6700 2500
-F 0 "#PWR015" H 6700 2350 50  0001 C CNN
-F 1 "+3.3V" V 6700 2750 50  0000 C CNN
-F 2 "" H 6700 2500 50  0001 C CNN
-F 3 "" H 6700 2500 50  0001 C CNN
-	1    6700 2500
+P 6400 2500
+F 0 "#PWR015" H 6400 2350 50  0001 C CNN
+F 1 "+3.3V" V 6400 2750 50  0000 C CNN
+F 2 "" H 6400 2500 50  0001 C CNN
+F 3 "" H 6400 2500 50  0001 C CNN
+	1    6400 2500
 	0    -1   -1   0
 $EndComp
@@
 	2500 5725 2400 5725
 Wire Wire Line
-	6700 2500 6850 2500
+	6400 2500 6550 2500
 Text GLabel 7700 2500 2    60   Input ~ 0
 reset

Commit message: terminal footprints
Parts:
- J4, J5, J6: footprint Terminal:WAGO_2pin -> Terminal:Terminal_1x2_2.54mm
Changed lines of the file:
@@
 F 0 "J6" H 6800 1175 50  0000 C TNN
 F 1 "RND 205-00232" H 6525 1275 50  0000 C TNN
-F 2 "Terminal:WAGO_2pin" H 6725 1250 50  0001 C CNN
+F 2 "Terminal:Terminal_1x2_2.54mm" H 6725 1250 50  0001 C CNN
 F 3 "" H 6700 1475 50  0001 C CNN
 	1    6725 1475
@@
 F 0 "J5" H 3950 6000 50  0000 C TNN
 F 1 "RND 205-00232" H 3675 6075 50  0000 C TNN
-F 2 "Terminal:WAGO_2pin" H 3900 6050 50  0001 C CNN
+F 2 "Terminal:Terminal_1x2_2.54mm" H 3900 6050 50  0001 C CNN
 F 3 "" H 3875 6275 50  0001 C CNN
 	1    3900 6275
@@
 F 0 "J4" H 3950 5975 50  0000 C TNN
 F 1 "RND 205-00232" H 3675 5900 50  0000 C TNN
-F 2 "Terminal:WAGO_2pin" H 3900 5400 50  0001 C CNN
+F 2 "Terminal:Terminal_1x2_2.54mm" H 3900 5400 50  0001 C CNN
 F 3 "" H 3875 5625 50  0001 C CNN
 	1    3900 5625
